File: KiCad/jongseol_cad - 복사본/jongseol/_autosave-jongseol.kicad_sch (KiCad schematic)
At the start: 10 parts, among them J1 Power, J2 Analog, J3 Analog, J4 Digital, J5 PWM, J6 PWM, J7 Communication, U1 ultrasonic_sensor

Commit message: 2022-08-29_16:13:09.50
Parts:
- gave numbers to parts that had none: 1
Changed lines of the file:
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@@
   (symbol (lib_id "power:GND") (at 110.49 123.19 270) (unit 1)
     (in_bom yes) (on_board yes)
-    (property "Reference" "#PWR?" (id 0) (at 104.14 123.19 0)
+    (property "Reference" "#PWR012" (id 0) (at 104.14 123.19 0)
       (effects (font (size 1.27 1.27)) hide)
     )
@@
   (symbol (lib_id "power:+5V") (at 110.49 146.05 90) (unit 1)
     (in_bom yes) (on_board yes)
-    (property "Reference" "#PWR?" (id 0) (at 114.3 146.05 0)
+    (property "Reference" "#PWR013" (id 0) (at 114.3 146.05 0)
       (effects (font (size 1.27 1.27)) hide)
     )
@@
   (symbol (lib_id "My_Symbol:8_channel_relay") (at 113.03 121.92 0) (unit 1)
     (in_bom yes) (on_board yes) (fields_autoplaced)
-    (property "Reference" "R?" (id 0) (at 119.38 133.3499 0)
+    (property "Reference" "R1" (id 0) (at 119.38 133.3499 0)
       (effects (font (size 1.27 1.27)) (justify left))
     )
@@
     )
     (path "/358c03c9-9a4f-4366-b762-cafd1c5870f6"
-      (reference "#PWR?") (unit 1) (value "GND") (footprint "")
+      (reference "#PWR012") (unit 1) (value "GND") (footprint "")
     )
     (path "/a405ec44-e794-49b9-8084-aaa4d6f0bec2"
-      (reference "#PWR?") (unit 1) (value "+5V") (footprint "")
+      (reference "#PWR013") (unit 1) (value "+5V") (footprint "")
     )
     (path "/2186f868-11e1-407e-8b52-aaf674efb8f2"
@@
     )
     (path "/dd4217a1-6732-48bb-ac15-01dbaea2d68a"
-      (reference "R?") (unit 1) (value "8_channel_relay") (footprint "My_Lib:8_channel_relay")
+      (reference "R1") (unit 1) (value "8_channel_relay") (footprint "My_Lib:8_channel_relay")
     )
     (path "/e8312ae2-495e-410d-844e-b1c4504481e0"
