File: KiCad/jongseol_cad/jongseol/jongseol.kicad_sch (KiCad schematic)
At the start: 10 parts, among them J1 Power, J2 Analog, J3 Analog, J4 Digital, J5 PWM, J6 PWM, J7 Communication, U1 ultrasonic_sensor

Commit message: 2022-09-05_17:31:53.18
Parts:
- added B1: MH_FMD_Buzzer, My_Lib:MH_FMD_Buzzer, symbol My_Symbol:MH_FMD_Buzzer
- gave numbers to parts that had none: 1
Connections:
- net +5V: now also B1.3 (VCC)
- net GND: now also B1.1 (GND)
- net *10 renamed Buzzer
- net Buzzer: now also B1.2 (I/O)
Other:
- moved on the sheet: R1, U1
