File: KiCad/jongseol_cad/jongseol/jongseol.kicad_pcb (KiCad board)
At the start: 2 copper layers, 101.6 x 53.3 mm, 13 parts, among them J1 Power, J2 PWM, J3 Analog, J4 PWM, J5 Analog, J6 Communication, J7 Digital

Commit message: 2022-08-29_16:13:09.50
Parts:
- removed MH4: MountingHole_3.2mm, Arduino_MountingHole:MountingHole_3.2mm
- added E1: ESP32, My_Lib:ESP32, F.Cu at (120.1, 88.4)
- added Relay: 8_channel_relay, My_Lib:8_channel_relay, F.Cu at (146.1, 94.4)
- added Ultrasonic: ultrasonic_sensor, My_Lib:ultrasonic_sensor, F.Cu at (127.7, 59.4)
- renumbered J3 to J2, J5 to J3, J7 to J4, J2 to J5, J4 to J6, J6 to J7
Connections:
- J2 pad 1: /A0 -> Relay_1
- J2 pad 2: /A1 -> Relay_2
- J2 pad 3: /A2 -> Relay_3
- J2 pad 4: /A3 -> Relay_4
- J2 pad 5: /A4 -> Relay_5
- J2 pad 6: /A5 -> Relay_6
- J2 pad 7: /A6 -> Relay_7
- J2 pad 8: /A7 -> Relay_8
- J5 pad 10: /*8 -> Echo
- J5 pad 9: /*9 -> Trig
- J6 pad 7: /TX0/1 -> TX
- J6 pad 8: /RX0/0 -> RX
Routing:
- net +5V: track 0.00 -> 162.3 mm
- net /SCL/21: track 0.00 -> 72.4 mm
- net /SDA/20: track 0.00 -> 66.5 mm
- net RX: track 0.00 -> 32.8 mm
- net TX: track 0.00 -> 28.1 mm, vias 0 -> 1
- net Trig: track 0.00 -> 10.3 mm
- net Echo: track 0.00 -> 10.3 mm
- net Relay_8: track 0.00 -> 5.72 mm
- net Relay_7: track 0.00 -> 5.72 mm
- net Relay_6: track 0.00 -> 5.72 mm
- net Relay_5: track 0.00 -> 5.72 mm
- net Relay_4: track 0.00 -> 5.72 mm
- net Relay_3: track 0.00 -> 5.72 mm
- net Relay_2: track 0.00 -> 5.72 mm
- net Relay_1: track 0.00 -> 5.72 mm
- added copper zone on B.Cu, net GND
Other:
- outline, holes or cut-outs redrawn
- board text removed: "ICSP"

Commit message: 2022-09-05_17:31:53.18
Parts:
- added B1: Buzzer, My_Lib:MH_FMD_Buzzer, F.Cu at (120.1, 59.4)
- E1: value ESP32 -> ESP32-CAM
- R1: renamed from Relay; value 8_channel_relay -> Relay
- U1: renamed from Ultrasonic; value ultrasonic_sensor -> Ultrasonic
- moved R1 30.8 mm to (115.9, 88.5), turned to 180 degrees
- moved U1 4.10 mm to (131.8, 59.4)
Connections:
- J5 pad 8: /*10 -> Buzzer
Routing:
- net Relay_8: track 5.72 -> 77.8 mm
- net Relay_7: track 5.72 -> 73.5 mm
- net Relay_6: track 5.72 -> 69.4 mm
- net Relay_5: track 5.72 -> 64.8 mm
- net Relay_4: track 5.72 -> 60.4 mm
- net Relay_3: track 5.72 -> 56.1 mm
- net Relay_2: track 5.72 -> 51.8 mm
- net Relay_1: track 5.72 -> 47.4 mm
- net +5V: track 162.3 -> 201.3 mm
- net Buzzer: track 0.00 -> 16.1 mm
- net Trig: track 10.3 -> 8.53 mm
- net Echo: track 10.3 -> 8.53 mm
- net TX: vias 1 -> 2
Other:
- board size 101.6 x 53.3 mm -> 91.6 x 53.3 mm

Commit message: 2022-09-06_17:31:50.91
Parts:
- added Display1: DM43, My_Lib:DM43_LCD_Module, F.Cu at (162.8, 54.3)
- B1: value Buzzer -> MH_FMD
- E1: value ESP32-CAM -> ESP32
- moved U1 1.52 mm to (133.4, 59.4)
Connections:
- net /SCL/21 renamed SCL
- net /SDA/20 renamed SDA
Routing:
- net +5V: track 201.3 -> 236.0 mm
- net SCL: track 72.4 -> 76.7 mm
- net SDA: track 66.5 -> 70.7 mm, vias 0 -> 1
- net RX: track 32.8 -> 34.4 mm
- net TX: track 28.1 -> 29.4 mm, vias 2 -> 1
- net Trig: track 8.53 -> 7.90 mm
- net Echo: track 8.53 -> 7.90 mm
