File: KiCad/jonseol2/jonseol2.kicad_pcb (KiCad board)
At the start: 2 copper layers, 90.9 x 66 mm, 21 parts, among them J1 Power, J2 Analog, J3 Analog, J4 Digital, J5 PWM, J6 PWM, J7 Communication, U1 Ultrasonic

Commit message: 2022-09-06_23:20:56.56
Parts:
- Display1: value DM43 -> LCD
Changed lines of the file:
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@@
     (grid_origin 100 100)
     (pcbplotparams
-      (layerselection 0x0000030_80000001)
+      (layerselection 0x0000030_ffffffff)
       (disableapertmacros false)
       (usegerberextensions false)
@@
       (outputformat 1)
       (mirror false)
-      (drillshape 1)
+      (drillshape 0)
       (scaleselection 1)
-      (outputdirectory "")
+      (outputdirectory "gerber/")
     )
   )
@@
       (effects (font (size 1 1) (thickness 0.15)))
     )
-    (fp_text value "DM43" (at 2.484 -2.745 unlocked) (layer "F.SilkS")
+    (fp_text value "LCD" (at 2.484 -2.745 unlocked) (layer "F.SilkS")
       (effects (font (size 1 1) (thickness 0.15)))
     )
@@
       (effects (font (size 1 1) (thickness 0.15)))
     )
-    (fp_text value "Relay" (at 2.54 29.21 90 unlocked) (layer "F.Fab")
-      (effects (font (size 1 1) (thickness 0.15)))
-    )
+    (fp_text value "Relay" (at 2.54 -2.54 unlocked) (layer "F.SilkS")
+      (effects (font (size 1 1) (thickness 0.15)))
+    )

Commit message: 2022-09-07_15:03:23.49
Routing:
- net +5V: track 0.00 -> 68.1 mm
- net VCC: track 18.9 -> 0.00 mm
